File: eeg-wings.sch (KiCad schematic (older format))
At the start: 3 parts

Commit message: schematic almost done
Parts:
- removed U?: ADS1299, Package_QFP:TQFP-64_10x10mm_P0.5mm, symbol Analog_ADC:ADS1298xPAG
- added C? (x6): 10uF, symbol Device:C_Small
- added C?: 10nF, symbol Device:C_Small
- added U1: LM2664, symbol mine:LM2664
- added U2: MCP1754-3302E_SOT89, Package_TO_SOT_SMD:SOT-89-3, symbol Regulator_Linear:MCP1754-3302E_SOT89
- added U3: TLV70025_SOT23-5, Package_TO_SOT_SMD:SOT-23-5, symbol Regulator_Linear:TLV70025_SOT23-5
- added U4: TPS72325_SOT23-5, Package_TO_SOT_SMD:SOT-23-5, symbol mine:TPS72325_SOT23-5
- J1: renamed from J?; value Conn_01x16_Female -> Adafruit Wing Header Left; footprint (none) -> Connector_PinSocket_2.54mm:PinSocket_1x16_P2.54mm_Vertical
- J2: renamed from J?; value Conn_01x12_Female -> Adafruit Wing Header Right; footprint (none) -> Connector_PinSocket_2.54mm:PinSocket_1x12_P2.54mm_Vertical
Connections:
- net labels added: +2.5V, -2.5V, -3.3V, D1, D2, D3, D4, D5, D6, D7, GNDA, NC, PWDN, RESET, SCLK, SDA, SDL, VDD, VDDA, VSSA
- net labels removed: DFU
- wire segments 28 -> 50
- no-connect marks 0 -> 6
Other:
- note added: "3.3V Regulator"
- note added: "Negative Regulator"
- note added: "Positive Regulator"
- note added: "Voltage Inverter"
- moved on the sheet: J1, J2
