File: eeg-wings.sch (KiCad schematic (older format))
At the start: 13 parts, among them J1 Adafruit Wing Header Left, J2 Adafruit Wing Header Right, U1 LM2664, U2 MCP1754-3302E_SOT89, U3 TLV70025_SOT23-5, U4 TPS72325_SOT23-5

Commit message: schematic
Parts:
- gave numbers to parts that had none: 7
Changed lines of the file:
@@
 Rev ""
 Comp "openlabs.co"
-Comment1 "Thomas Stilwell / Maryjane Cook"
-Comment2 "stilwellt@openlabs.co"
-Comment3 ""
+Comment1 "stilwellt@openlabs.co"
+Comment2 "Thomas Stilwell"
+Comment3 "Maryjane Cook"
 Comment4 ""
 $EndDescr
@@
 	6400 3100 7450 3100
 $Comp
-L Device:C_Small C?
+L Device:C_Small C27
 U 1 1 5FEEEFFA
 P 1150 6600
-F 0 "C?" H 1059 6554 50  0000 R CNN
+F 0 "C27" H 1059 6554 50  0000 R CNN
 F 1 "10uF" H 1059 6645 50  0000 R CNN
 F 2 "" H 1150 6600 50  0001 C CNN
@@
 Connection ~ 1900 6500
 $Comp
-L Device:C_Small C?
+L Device:C_Small C29
 U 1 1 5FEF2C7D
 P 2300 7000
-F 0 "C?" H 2209 6954 50  0000 R CNN
+F 0 "C29" H 2209 6954 50  0000 R CNN
 F 1 "10uF" H 2209 7045 50  0000 R CNN
 F 2 "" H 2300 7000 50  0001 C CNN
@@
 	2300 6900 3300 6900
 $Comp
-L power:GNDA #PWR?
+L power:GNDA #PWR0101
 U 1 1 5FEF3059
 P 2300 7100
-F 0 "#PWR?" H 2300 6850 50  0001 C CNN
+F 0 "#PWR0101" H 2300 6850 50  0001 C CNN
 F 1 "GNDA" H 2305 6927 50  0000 C CNN
 F 2 "" H 2300 7100 50  0001 C CNN
@@
 Connection ~ 3300 6900
 $Comp
-L Device:C_Small C?
+L Device:C_Small C30
 U 1 1 5FEFA71E
 P 2450 5050
-F 0 "C?" H 2359 5004 50  0000 R CNN
+F 0 "C30" H 2359 5004 50  0000 R CNN
 F 1 "10uF" H 2359 5095 50  0000 R CNN
 F 2 "" H 2450 5050 50  0001 C CNN
@@
 	2450 4950 2600 4950
 $Comp
-L power:GNDA #PWR?
+L power:GNDA #PWR0168
 U 1 1 5FEFAA47
 P 2450 5150
-F 0 "#PWR?" H 2450 4900 50  0001 C CNN
+F 0 "#PWR0168" H 2450 4900 50  0001 C CNN
 F 1 "GNDA" H 2455 4977 50  0000 C CNN
 F 2 "" H 2450 5150 50  0001 C CNN
@@
 $EndComp
 $Comp
-L Device:C_Small C?
+L Device:C_Small C31
 U 1 1 5FEFB04A
 P 3850 5050
-F 0 "C?" H 3758 5004 50  0000 R CNN
+F 0 "C31" H 3758 5004 50  0000 R CNN
 F 1 "10uF" H 3758 5095 50  0000 R CNN
 F 2 "" H 3850 5050 50  0001 C CNN
@@
 	3850 4950 3800 4950
 $Comp
-L power:GNDA #PWR?
+L power:GNDA #PWR0169
 U 1 1 5FEFB65C
 P 3850 5150
-F 0 "#PWR?" H 3850 4900 50  0001 C CNN
+F 0 "#PWR0169" H 3850 4900 50  0001 C CNN
 F 1 "GNDA" H 3855 4977 50  0000 C CNN
 F 2 "" H 3850 5150 50  0001 C CNN
@@
 $EndComp
 $Comp
-L Device:C_Small C?
+L Device:C_Small C33
 U 1 1 5FEFB82B
 P 4250 7000
-F 0 "C?" H 4158 6954 50  0000 R CNN
+F 0 "C33" H 4158 6954 50  0000 R CNN
 F 1 "10uF" H 4158 7045 50  0000 R CNN
 F 2 "" H 4250 7000 50  0001 C CNN
@@
 	4250 6900 3900 6900
 $Comp
-L power:GNDA #PWR?
+L power:GNDA #PWR0170
 U 1 1 5FEFBAB1
 P 4250 7100
-F 0 "#PWR?" H 4250 6850 50  0001 C CNN
+F 0 "#PWR0170" H 4250 6850 50  0001 C CNN
 F 1 "GNDA" H 4255 6927 50  0000 C CNN
 F 2 "" H 4250 7100 50  0001 C CNN
@@
 $EndComp
 $Comp
-L Device:C_Small C?
+L Device:C_Small C32
 U 1 1 5FEFBC80
 P 3900 7150
-F 0 "C?" H 3808 7104 50  0000 R CNN
+F 0 "C32" H 3808 7104 50  0000 R CNN
 F 1 "10nF" H 3808 7195 50  0000 R CNN
 F 2 "" H 3900 7150 50  0001 C CNN
@@
 $EndComp
 $Comp
-L power:GNDA #PWR?
+L power:GNDA #PWR0171
 U 1 1 5FEFBE47
 P 3900 7250
-F 0 "#PWR?" H 3900 7000 50  0001 C CNN
+F 0 "#PWR0171" H 3900 7000 50  0001 C CNN
 F 1 "GNDA" H 3905 7077 50  0000 C CNN
 F 2 "" H 3900 7250 50  0001 C CNN
@@
 $EndComp
 $Comp
-L Device:C_Small C?
+L Device:C_Small C28
 U 1 1 5FEFDDAB
 P 1450 5050
-F 0 "C?" H 1250 5100 50  0000 L CNN
+F 0 "C28" H 1250 5100 50  0000 L CNN
 F 1 "10uF" H 1150 5000 50  0000 L CNN
 F 2 "" H 1450 5050 50  0001 C CNN
@@
 	1150 4950 1450 4950
 $Comp
-L power:GNDA #PWR?
+L power:GNDA #PWR0172
 U 1 1 5FF02E07
 P 1450 5150
-F 0 "#PWR?" H 1450 4900 50  0001 C CNN
+F 0 "#PWR0172" H 1450 4900 50  0001 C CNN
 F 1 "GNDA" H 1455 4977 50  0000 C CNN
 F 2 "" H 1450 5150 50  0001 C CNN
