File: Analog-Left.sch (KiCad schematic (older format))
At the start: 30 parts, among them J3 Conn_01x13, J4 Conn_01x13, U5 ADS1299

Commit message: schematic
Parts:
- removed R1, R2, R3, R4: 2k2, symbol Device:R_Small
- removed RN1, RN2: 2k2, symbol Device:R_Pack08
- added RN1: 2k2, Resistor_SMD:R_Array_Concave_4x0603, symbol Device:R_Pack04_Split
- added RN2, RN3, RN4, RN5: 2k2, Resistor_SMD:R_Array_Concave_4x0603, symbol Device:R_Pack04
- C1, C2, C3, C4, C5, C6: value C_4_Small -> 1nF; footprint (none) -> Resistor_SMD:R_Array_Concave_4x0603
- C10, C11, C12, C13, C8, C9: footprint (none) -> Capacitor_SMD:C_0603_1608Metric
- C7: value C_Small -> 1nF; footprint (none) -> Capacitor_SMD:C_0603_1608Metric
- D1, D2, D3, D4, D5, D6: footprint (none) -> Package_TO_SOT_SMD:SC-70-8
- R5: value R_Small -> 1M; footprint (none) -> Resistor_SMD:R_0603_1608Metric
- R6: footprint (none) -> Resistor_SMD:R_0603_1608Metric
Connections:
- net 1N: now also RN5.3 (R3.1)
- net 1P: now also RN3.3 (R3.1)
- net 2N: now also RN5.2 (R2.1)
- net 2P: now also RN3.2 (R2.1)
- net 3N: now also RN5.1 (R1.1)
- net 3P: now also RN3.1 (R1.1)
- net 4N: now also RN4.4 (R4.1)
- net 4P: now also RN2.4 (R4.1)
- net 5N: now also RN4.3 (R3.1)
- net 5P: now also RN2.3 (R3.1)
- net 6N: now also RN4.2 (R2.1)
- net 6P: now also RN2.2 (R2.1)
- net 7N: now also RN4.1 (R1.1)
- net 7P: now also RN2.1 (R1.1)
- net 8N: now also RN1.4
- net 8P: now also RN1.2
- net BIAS: now also RN1.1, RN1.3
- net BIAS_DRV: now also RN1.6, RN1.8
- net GND: now also U5.60 (BIASREF); no longer C1.3, C2.3
- net SRB1: now also RN3.4 (R4.1)
- net SRB2: now also RN5.4 (R4.1)
- net at C4.5, U5.12 (IN3P): now also RN3.8 (R1.2)
- net at C4.6, U5.14 (IN2P): now also RN3.7 (R2.2)
- net at C4.7, U5.16 (IN1P): now also RN3.6 (R3.2)
- net at C4.8, U5.17 (SRB1): now also RN3.5 (R4.2)
- net at C3.5, U5.3 (IN7P): now also RN2.8 (R1.2)
- net at C3.6, U5.6 (IN6P): now also RN2.7 (R2.2)
- net at C3.7, U5.8 (IN5P): now also RN2.6 (R3.2)
- net at C3.8, U5.10 (IN4P): now also RN2.5 (R4.2)
- net at C1.1, U5.2 (IN8P): now also RN1.7
- net at C5.5, U5.11 (IN3N): now also RN5.8 (R1.2)
- net at C5.6, U5.13 (IN2N): now also RN5.7 (R2.2)
- net at C5.7, U5.15 (IN1N): now also RN5.6 (R3.2)
- net at C5.8, U5.18 (SRB2): now also RN5.5 (R4.2)
- net at C6.5, U5.4 (IN7N): now also RN4.8 (R1.2)
- net at C6.6, U5.5 (IN6N): now also RN4.7 (R2.2)
- net at C6.7, U5.7 (IN5N): now also RN4.6 (R3.2)
- net at C6.8, U5.9 (IN4N): now also RN4.5 (R4.2)
- net at C2.1, U5.1 (IN8N): now also RN1.5
- no-connect marks 3 -> 6

Commit message: dunno
Parts:
- removed C1: 1nF, Resistor_SMD:R_Array_Concave_4x0603, symbol mine:C_4_Small
- removed D2: D_TVS_4, Package_TO_SOT_SMD:SC-70-8, symbol mine:D_TVS_4
- D1, D3, D4, D5, D6: footprint Package_TO_SOT_SMD:SC-70-8 -> Package_TO_SOT_SMD:SOT-23-6
Connections:
- net 1N: now also D1.2; no longer D1.4
- net 1P: now also D3.2; no longer D3.4
- net 3N: now also D1.4; no longer D6.1
- net 3P: now also D3.4; no longer D4.1
- net 4N: now also D6.1; no longer D6.2
- net 4P: now also D4.1; no longer D4.2
- net 5N: now also D6.2; no longer D6.4
- net 5P: now also D4.2; no longer D4.4
- net 7N: now also D6.4; no longer D5.5
- net 7P: now also D4.4
- net 8N: now also D5.1; no longer D5.4
- net 8P: now also D5.5
- net BIAS: now also D5.4
- net BIAS_DRV: now also C2.1, C2.3; no longer C2.2
- net SRB1: now also D3.1; no longer D3.2
- net SRB2: now also D1.1; no longer D1.2
- net VDDA: no longer D5.1
- net VSSA: no longer D1.1, D3.1
- net 8PA: now reaches RN1.7, U5.2 (IN8P)
- net 8PA: now also C2.2
- net at RN1.5, U5.1 (IN8N): now also C2.4; no longer C2.1
- no-connect marks 6 -> 2
Other:
- moved on the sheet: C16, D10
