File: eeg-wings.kicad_pcb (KiCad board)
At the start: 2 copper layers, 50.8 x 22.9 mm, 15 parts, among them J1 Adafruit Wing Header Left, J2 Adafruit Wing Header Right, J3 Conn_01x13, J4 Conn_01x13, J5 Conn_01x13, J6 Conn_01x13, U2 MCP1754-3302E_SOT89, U3 TLV70025_SOT23-5, U4 TPS72325_SOT23-5, U5 ADS1299, U6 ADS1299

Commit message: schematic
Parts:
- added C1: 1nF, Resistor_SMD:R_Array_Concave_4x0603, F.Cu at (111.4, 83.4)
- added C10: 1uF, Capacitor_SMD:C_0603_1608Metric, F.Cu at (132.1, 113.8)
- added C11: 100uF, Capacitor_SMD:C_0603_1608Metric, F.Cu at (127.0, 114.3)
- added C12: 0.1uF, Capacitor_SMD:C_0603_1608Metric, F.Cu at (130.8, 91.0)
- added C13: 1uF, Capacitor_SMD:C_0603_1608Metric, F.Cu at (127.0, 88.9)
- added C14: 1nF, Resistor_SMD:R_Array_Concave_4x0603, F.Cu at (187.9, 94.7)
- added C15: 1nF, Resistor_SMD:R_Array_Concave_4x0603, F.Cu at (187.2, 117.5)
- added C16: 1nF, Resistor_SMD:R_Array_Concave_4x0603, F.Cu at (181.6, 121.9)
- added C17: 1nF, Resistor_SMD:R_Array_Concave_4x0603, F.Cu at (187.9, 111.6)
- added C18: 1nF, Resistor_SMD:R_Array_Concave_4x0603, F.Cu at (187.7, 106.3)
- added C19: 1nF, Resistor_SMD:R_Array_Concave_4x0603, F.Cu at (187.8, 100.6)
- added C2: 1nF, Resistor_SMD:R_Array_Concave_4x0603, F.Cu at (114.3, 74.9)
- added C20: 1nF, Capacitor_SMD:C_0603_1608Metric, F.Cu at (175.3, 117.6)
- added C21: 10uF, Capacitor_SMD:C_0603_1608Metric, F.Cu at (172.7, 88.1)
- added C22: 1uF, Capacitor_SMD:C_0603_1608Metric, F.Cu at (170.2, 85.6)
- added C23: 1uF, Capacitor_SMD:C_0603_1608Metric, F.Cu at (165.1, 81.3)
- added C24: 100uF, Capacitor_SMD:C_0603_1608Metric, F.Cu at (165.1, 88.9)
- added C25: 0.1uF, Capacitor_SMD:C_0603_1608Metric, F.Cu at (167.6, 125.7)
- added C26: 1uF, Capacitor_SMD:C_0603_1608Metric, F.Cu at (168.9, 116.1)
- added C3: 1nF, Resistor_SMD:R_Array_Concave_4x0603, F.Cu at (117.2, 111.3)
- added C4: 1nF, Resistor_SMD:R_Array_Concave_4x0603, F.Cu at (112.6, 116.0)
- added C5: 1nF, Resistor_SMD:R_Array_Concave_4x0603, F.Cu at (110.9, 108.4)
- added C6: 1nF, Resistor_SMD:R_Array_Concave_4x0603, F.Cu at (115.2, 89.3)
- added C7: 1nF, Capacitor_SMD:C_0603_1608Metric, F.Cu at (121.9, 86.4)
- added C8: 10uF, Capacitor_SMD:C_0603_1608Metric, F.Cu at (123.2, 118.6)
- added C9: 1uF, Capacitor_SMD:C_0603_1608Metric, F.Cu at (123.2, 112.2)
- added R11: 1M, Resistor_SMD:R_0603_1608Metric, F.Cu at (172.7, 116.8)
- added R12: 10k, Resistor_SMD:R_0603_1608Metric, F.Cu at (165.1, 116.8)
- added R5: 1M, Resistor_SMD:R_0603_1608Metric, F.Cu at (121.9, 80.0)
- added R6: 10k, Resistor_SMD:R_0603_1608Metric, F.Cu at (125.7, 78.7)
- added RN1: 2k2, Resistor_SMD:R_Array_Concave_4x0603, F.Cu at (105.4, 91.4)
- added RN10: 2k2, Resistor_SMD:R_Array_Concave_4x0603, F.Cu at (191.8, 111.8)
- added RN2: 2k2, Resistor_SMD:R_Array_Concave_4x0603, F.Cu at (113.0, 102.9)
- added RN3: 2k2, Resistor_SMD:R_Array_Concave_4x0603, F.Cu at (105.4, 111.8)
- added RN4: 2k2, Resistor_SMD:R_Array_Concave_4x0603, F.Cu at (113.0, 97.8)
- added RN5: 2k2, Resistor_SMD:R_Array_Concave_4x0603, F.Cu at (105.8, 107.1)
- added RN6: 2k2, Resistor_SMD:R_Array_Concave_4x0603, F.Cu at (192.0, 94.3)
- added RN7: 2k2, Resistor_SMD:R_Array_Concave_4x0603, F.Cu at (191.9, 106.2)
- added RN8: 2k2, Resistor_SMD:R_Array_Concave_4x0603, F.Cu at (191.8, 117.7)
- added RN9: 2k2, Resistor_SMD:R_Array_Concave_4x0603, F.Cu at (192.0, 100.8)
- moved J6 73.6 mm to (200.7, 88.9), turned to 0 degrees
- moved J5 68.4 mm to (196.8, 88.9), turned to 0 degrees
- moved J3 66.6 mm to (95.2, 83.8), turned to 0 degrees
- moved U4 63.8 mm to (148.6, 106.7), turned to 270 degrees
- moved J4 60.6 mm to (100.3, 83.8), turned to 0 degrees
- moved U3 53.4 mm to (148.6, 96.5), turned to 270 degrees
- moved U2 49.9 mm to (149.9, 86.4), turned to 270 degrees
- moved REF** 45.9 mm to (158.1, 125.7), turned to 270 degrees
- moved REF** 43.2 mm to (139.1, 125.7), turned to 270 degrees
- moved U6 38.6 mm to (170.2, 102.9), turned to 180 degrees
- moved U5 30.0 mm to (127.0, 101.6), turned to 0 degrees
- moved REF** 28.2 mm to (157.5, 80.0), turned to 270 degrees
- moved REF** 23.9 mm to (139.7, 80.0), turned to 270 degrees
- moved J1 19.7 mm to (138.4, 83.8), turned to 0 degrees
- moved J2 19.1 mm to (158.8, 94.0), turned to 0 degrees
Connections:
- net /DFU renamed /NC
- U4 pad 3: Net-(U4-Pad3) -> /-3.3V
- U5 pad 60: Net-(U5-Pad60) -> GND
- U6 pad 60: Net-(U6-Pad60) -> GND
Other:
- board size 50.8 x 22.9 mm -> 22.9 x 50.8 mm

Commit message: dunno
Parts:
- removed C1, C14: 1nF, Resistor_SMD:R_Array_Concave_4x0603
- added D1: D_TVS_4, Package_TO_SOT_SMD:SOT-23-6, F.Cu at (135.5, 65.0)
- added D10: D_TVS_4, Package_TO_SOT_SMD:SOT-23-6, F.Cu at (197.7, 116.5)
- added D11: D_TVS_4, Package_TO_SOT_SMD:SOT-23-6, F.Cu at (197.7, 104.4)
- added D12: D_TVS_4, Package_TO_SOT_SMD:SOT-23-6, F.Cu at (197.7, 110.8)
- added D3: D_TVS_4, Package_TO_SOT_SMD:SOT-23-6, F.Cu at (139.9, 65.0)
- added D4: D_TVS_4, Package_TO_SOT_SMD:SOT-23-6, F.Cu at (139.9, 68.7)
- added D5: D_TVS_4, Package_TO_SOT_SMD:SOT-23-6, F.Cu at (144.4, 65.0)
- added D6: D_TVS_4, Package_TO_SOT_SMD:SOT-23-6, F.Cu at (144.4, 68.7)
- added D7: D_TVS_4, Package_TO_SOT_SMD:SOT-23-6, F.Cu at (197.7, 92.0)
- added D8: D_TVS_4, Package_TO_SOT_SMD:SOT-23-6, F.Cu at (197.7, 98.0)
- moved J5 31.1 mm to (203.2, 119.4), turned to 180 degrees
- moved J6 30.9 mm to (205.7, 119.4), turned to 180 degrees
- moved RN8 25.7 mm to (192.5, 92.0), turned to 180 degrees
- moved C15 25.5 mm to (188.1, 92.0), turned to 0 degrees
- moved RN6 22.2 mm to (192.5, 116.5)
- moved RN10 13.8 mm to (192.5, 98.0), turned to 180 degrees
- moved C17 13.6 mm to (188.1, 98.0), turned to 0 degrees
- moved C19 10.2 mm to (188.1, 110.8)
- moved RN9 10.0 mm to (192.5, 110.8), turned to 180 degrees
- moved C16 8.46 mm to (188.1, 116.5), turned to 180 degrees
- moved U6 5.44 mm to (175.3, 104.7)
- moved C18 1.94 mm to (188.1, 104.4)
- moved RN7 1.90 mm to (192.5, 104.4), turned to 180 degrees
Connections:
- C15 pad 1: Net-(C15-Pad1) -> GND
- C15 pad 3: Net-(C15-Pad3) -> GND
- C15 pad 6: GND -> Net-(C15-Pad6)
- C15 pad 8: GND -> Net-(C15-Pad8)
- C16 pad 1: GND -> /Analog-Right/BIAS_DRV
- C16 pad 2: Net-(C16-Pad2) -> /Analog-Right/8PA
- C16 pad 3: GND -> /Analog-Right/BIAS_DRV
- C16 pad 4: /Analog-Right/BIAS_DRV -> Net-(C16-Pad4)
- C16 pad 6: Net-(C16-Pad6) -> GND
- C16 pad 8: Net-(C16-Pad8) -> GND
- C17 pad 1: Net-(C17-Pad1) -> GND
- C17 pad 3: Net-(C17-Pad3) -> GND
- C17 pad 6: GND -> Net-(C17-Pad6)
- C17 pad 8: GND -> Net-(C17-Pad8)
- C18 pad 1: Net-(C18-Pad1) -> GND
- C18 pad 3: Net-(C18-Pad3) -> GND
- C18 pad 6: GND -> Net-(C18-Pad6)
- C18 pad 8: GND -> Net-(C18-Pad8)
- C19 pad 1: Net-(C19-Pad1) -> GND
- C19 pad 3: Net-(C19-Pad3) -> GND
- C19 pad 6: GND -> Net-(C19-Pad6)
- C19 pad 8: GND -> Net-(C19-Pad8)
- C2 pad 1: GND -> /Analog-Left/BIAS_DRV
- C2 pad 2: Net-(C2-Pad2) -> /Analog-Left/8PA
- C2 pad 3: GND -> /Analog-Left/BIAS_DRV
- C2 pad 4: /Analog-Left/BIAS_DRV -> Net-(C2-Pad4)
- C2 pad 6: Net-(C2-Pad6) -> GND
- C2 pad 8: Net-(C2-Pad8) -> GND
- C3 pad 1: Net-(C3-Pad1) -> GND
- C3 pad 3: Net-(C3-Pad3) -> GND
- C3 pad 6: GND -> Net-(C3-Pad6)
- C3 pad 8: GND -> Net-(C3-Pad8)
- C4 pad 1: Net-(C4-Pad1) -> GND
- C4 pad 3: Net-(C4-Pad3) -> GND
- C4 pad 6: GND -> Net-(C4-Pad6)
- C4 pad 8: GND -> Net-(C4-Pad8)
- C5 pad 1: Net-(C5-Pad1) -> GND
- C5 pad 3: Net-(C5-Pad3) -> GND
- C5 pad 6: GND -> Net-(C5-Pad6)
- C5 pad 8: GND -> Net-(C5-Pad8)
- C6 pad 1: Net-(C6-Pad1) -> GND
- C6 pad 3: Net-(C6-Pad3) -> GND
- C6 pad 6: GND -> Net-(C6-Pad6)
- C6 pad 8: GND -> Net-(C6-Pad8)
- RN1 pad 5: Net-(C2-Pad2) -> Net-(C2-Pad4)
- RN1 pad 7: Net-(C1-Pad2) -> /Analog-Left/8PA
- RN10 pad 1: Net-(C17-Pad7) -> /Analog-Right/3N
- RN10 pad 2: Net-(C17-Pad5) -> /Analog-Right/2N
- RN10 pad 3: Net-(C17-Pad3) -> /Analog-Right/1N
- RN10 pad 4: Net-(C17-Pad1) -> /Analog-Right/SRB2
- RN10 pad 5: /Analog-Right/SRB2 -> Net-(C17-Pad8)
- RN10 pad 6: /Analog-Right/1N -> Net-(C17-Pad7)
- RN10 pad 7: /Analog-Right/2N -> Net-(C17-Pad6)
- RN10 pad 8: /Analog-Right/3N -> Net-(C17-Pad5)
- RN2 pad 1: Net-(C3-Pad7) -> /Analog-Left/7P
- RN2 pad 2: Net-(C3-Pad5) -> /Analog-Left/6P
- RN2 pad 3: Net-(C3-Pad3) -> /Analog-Left/5P
- RN2 pad 4: Net-(C3-Pad1) -> /Analog-Left/4P
- RN2 pad 5: /Analog-Left/4P -> Net-(C3-Pad8)
- RN2 pad 6: /Analog-Left/5P -> Net-(C3-Pad7)
- RN2 pad 7: /Analog-Left/6P -> Net-(C3-Pad6)
- RN2 pad 8: /Analog-Left/7P -> Net-(C3-Pad5)
- RN3 pad 1: Net-(C4-Pad7) -> /Analog-Left/3P
- RN3 pad 2: Net-(C4-Pad5) -> /Analog-Left/2P
- RN3 pad 3: Net-(C4-Pad3) -> /Analog-Left/1P
- RN3 pad 4: Net-(C4-Pad1) -> /Analog-Left/SRB1
- RN3 pad 5: /Analog-Left/SRB1 -> Net-(C4-Pad8)
- RN3 pad 6: /Analog-Left/1P -> Net-(C4-Pad7)
- RN3 pad 7: /Analog-Left/2P -> Net-(C4-Pad6)
- RN3 pad 8: /Analog-Left/3P -> Net-(C4-Pad5)
- RN4 pad 1: Net-(C6-Pad7) -> /Analog-Left/7N
- RN4 pad 2: Net-(C6-Pad5) -> /Analog-Left/6N
- RN4 pad 3: Net-(C6-Pad3) -> /Analog-Left/5N
- RN4 pad 4: Net-(C6-Pad1) -> /Analog-Left/4N
- RN4 pad 5: /Analog-Left/4N -> Net-(C6-Pad8)
- RN4 pad 6: /Analog-Left/5N -> Net-(C6-Pad7)
- RN4 pad 7: /Analog-Left/6N -> Net-(C6-Pad6)
- RN4 pad 8: /Analog-Left/7N -> Net-(C6-Pad5)
- RN5 pad 1: Net-(C5-Pad7) -> /Analog-Left/3N
- RN5 pad 2: Net-(C5-Pad5) -> /Analog-Left/2N
- RN5 pad 3: Net-(C5-Pad3) -> /Analog-Left/1N
- RN5 pad 4: Net-(C5-Pad1) -> /Analog-Left/SRB2
- RN5 pad 5: /Analog-Left/SRB2 -> Net-(C5-Pad8)
- RN5 pad 6: /Analog-Left/1N -> Net-(C5-Pad7)
- RN5 pad 7: /Analog-Left/2N -> Net-(C5-Pad6)
- RN5 pad 8: /Analog-Left/3N -> Net-(C5-Pad5)
- RN6 pad 5: Net-(C16-Pad2) -> Net-(C16-Pad4)
- RN6 pad 7: Net-(C14-Pad2) -> /Analog-Right/8PA
- RN7 pad 1: Net-(C18-Pad7) -> /Analog-Right/7P
- RN7 pad 2: Net-(C18-Pad5) -> /Analog-Right/6P
- RN7 pad 3: Net-(C18-Pad3) -> /Analog-Right/5P
- RN7 pad 4: Net-(C18-Pad1) -> /Analog-Right/4P
- RN7 pad 5: /Analog-Right/4P -> Net-(C18-Pad8)
- RN7 pad 6: /Analog-Right/5P -> Net-(C18-Pad7)
- RN7 pad 7: /Analog-Right/6P -> Net-(C18-Pad6)
- RN7 pad 8: /Analog-Right/7P -> Net-(C18-Pad5)
- RN8 pad 1: Net-(C15-Pad7) -> /Analog-Right/3P
- RN8 pad 2: Net-(C15-Pad5) -> /Analog-Right/2P
- RN8 pad 3: Net-(C15-Pad3) -> /Analog-Right/1P
- RN8 pad 4: Net-(C15-Pad1) -> /Analog-Right/SRB1
- RN8 pad 5: /Analog-Right/SRB1 -> Net-(C15-Pad8)
- RN8 pad 6: /Analog-Right/1P -> Net-(C15-Pad7)
- RN8 pad 7: /Analog-Right/2P -> Net-(C15-Pad6)
- RN8 pad 8: /Analog-Right/3P -> Net-(C15-Pad5)
- RN9 pad 1: Net-(C19-Pad7) -> /Analog-Right/7N
- RN9 pad 2: Net-(C19-Pad5) -> /Analog-Right/6N
- RN9 pad 3: Net-(C19-Pad3) -> /Analog-Right/5N
- RN9 pad 4: Net-(C19-Pad1) -> /Analog-Right/4N
- RN9 pad 5: /Analog-Right/4N -> Net-(C19-Pad8)
- RN9 pad 6: /Analog-Right/5N -> Net-(C19-Pad7)
- RN9 pad 7: /Analog-Right/6N -> Net-(C19-Pad6)
- RN9 pad 8: /Analog-Right/7N -> Net-(C19-Pad5)
- U5 pad 1: Net-(C2-Pad2) -> Net-(C2-Pad4)
- U5 pad 10: Net-(C3-Pad1) -> Net-(C3-Pad8)
- U5 pad 11: Net-(C5-Pad7) -> Net-(C5-Pad5)
- U5 pad 12: Net-(C4-Pad7) -> Net-(C4-Pad5)
- U5 pad 13: Net-(C5-Pad5) -> Net-(C5-Pad6)
- U5 pad 14: Net-(C4-Pad5) -> Net-(C4-Pad6)
- U5 pad 15: Net-(C5-Pad3) -> Net-(C5-Pad7)
- U5 pad 16: Net-(C4-Pad3) -> Net-(C4-Pad7)
- U5 pad 17: Net-(C4-Pad1) -> Net-(C4-Pad8)
- U5 pad 18: Net-(C5-Pad1) -> Net-(C5-Pad8)
- U5 pad 2: Net-(C1-Pad2) -> /Analog-Left/8PA
- U5 pad 3: Net-(C3-Pad7) -> Net-(C3-Pad5)
- U5 pad 4: Net-(C6-Pad7) -> Net-(C6-Pad5)
- U5 pad 5: Net-(C6-Pad5) -> Net-(C6-Pad6)
- U5 pad 6: Net-(C3-Pad5) -> Net-(C3-Pad6)
- U5 pad 7: Net-(C6-Pad3) -> Net-(C6-Pad7)
- U5 pad 8: Net-(C3-Pad3) -> Net-(C3-Pad7)
- U5 pad 9: Net-(C6-Pad1) -> Net-(C6-Pad8)
- U6 pad 1: Net-(C16-Pad2) -> Net-(C16-Pad4)
- U6 pad 10: Net-(C18-Pad1) -> Net-(C18-Pad8)
- U6 pad 11: Net-(C17-Pad7) -> Net-(C17-Pad5)
- U6 pad 12: Net-(C15-Pad7) -> Net-(C15-Pad5)
- U6 pad 13: Net-(C17-Pad5) -> Net-(C17-Pad6)
- U6 pad 14: Net-(C15-Pad5) -> Net-(C15-Pad6)
- U6 pad 15: Net-(C17-Pad3) -> Net-(C17-Pad7)
- U6 pad 16: Net-(C15-Pad3) -> Net-(C15-Pad7)
- U6 pad 17: Net-(C15-Pad1) -> Net-(C15-Pad8)
- U6 pad 18: Net-(C17-Pad1) -> Net-(C17-Pad8)
- U6 pad 2: Net-(C14-Pad2) -> /Analog-Right/8PA
- U6 pad 3: Net-(C18-Pad7) -> Net-(C18-Pad5)
- U6 pad 4: Net-(C19-Pad7) -> Net-(C19-Pad5)
- U6 pad 5: Net-(C19-Pad5) -> Net-(C19-Pad6)
- U6 pad 6: Net-(C18-Pad5) -> Net-(C18-Pad6)
- U6 pad 7: Net-(C19-Pad3) -> Net-(C19-Pad7)
- U6 pad 8: Net-(C18-Pad3) -> Net-(C18-Pad7)
- U6 pad 9: Net-(C19-Pad1) -> Net-(C19-Pad8)
Routing:
- net /Analog-Right/BIAS: track 0.00 -> 26.1 mm, vias 0 -> 1
- net /Analog-Right/SRB2: track 0.00 -> 15.7 mm, vias 0 -> 1
- net /Analog-Right/3P: track 0.00 -> 15.4 mm
- net /Analog-Right/8N: track 0.00 -> 15.4 mm
- net /Analog-Right/2N: track 0.00 -> 15.1 mm, vias 0 -> 1
- net /Analog-Right/1N: track 0.00 -> 15.0 mm, vias 0 -> 1
- net /Analog-Right/3N: track 0.00 -> 14.9 mm
- net /Analog-Right/2P: track 0.00 -> 14.6 mm
- net /Analog-Right/8P: track 0.00 -> 14.0 mm
- net /Analog-Right/1P: track 0.00 -> 12.8 mm
- net /Analog-Right/7P: track 0.00 -> 12.8 mm
- net /Analog-Right/6P: track 0.00 -> 12.7 mm
- net /Analog-Right/5P: track 0.00 -> 11.8 mm
- net /Analog-Right/SRB1: track 0.00 -> 11.4 mm
- net /Analog-Right/4P: track 0.00 -> 11.1 mm
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- added copper zone on In1.Cu, net GND
Other:
- copper layers 2 -> 4
- net class Default: via_dia 0.8 -> 0.6; via_drill 0.4 -> 0.3
